File: KiCad/Production/SenseU_Microphoneboard/SenseU_Microphoneboard.kicad_pcb (KiCad board)
At the start: 2 copper layers, 130 x 70.1 mm, 33 parts, among them J1 90122-0126

Commit message: Logo's
Parts:
- added G***: LOGO, LOGO, F.Cu at (138.4, 99.0)
- added kibuzzard-6486612E: G***, kibuzzard-6486612E, F.Cu at (136.7, 88.7)
- added kibuzzard-64866152: G***, kibuzzard-64866152, F.Cu at (130.1, 93.6)
- added kibuzzard-64904BCF: G***, kibuzzard-64904BCF, F.Cu at (135.1, 91.2)
