File: KiCad/Production/DisplayU_Sisterboard/_autosave-MCUnrf.kicad_sch (KiCad schematic)
At the start: 3 parts

Commit message: Microcontroller integration (almost done)
Parts:
- removed R1: 4.7k, symbol Device:R_Small
Connections:
- net MicroController/RST is gone; now on net VDD: RST.2 (B)
Changed lines of the file:
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@@
   (junction (at 68.58 116.84) (diameter 0) (color 0 0 0 0)
   )
-  (wire (pts (xy 68.58 111.125) (xy 68.58 111.76))
-    (stroke (width 0) (type default))
-  )
   (wire (pts (xy 130.175 78.74) (xy 146.05 78.74))
-    (stroke (width 0) (type default))
-  )
-  (wire (pts (xy 68.58 116.205) (xy 68.58 116.84))
     (stroke (width 0) (type default))
   )
@@
     (effects (font (size 1.27 1.27)) (justify left bottom))
   )
-  (hierarchical_label "GND" (shape input) (at 19.685 24.13 180) (fields_autoplaced)
+  (hierarchical_label "GND" (shape input) (at 42.545 84.455 180) (fields_autoplaced)
     (effects (font (size 1.27 1.27)) (justify right))
   )
-  (hierarchical_label "VDD" (shape input) (at 19.685 19.05 180) (fields_autoplaced)
+  (hierarchical_label "VDD" (shape input) (at 42.545 79.375 180) (fields_autoplaced)
     (effects (font (size 1.27 1.27)) (justify right))
   )
-  (hierarchical_label "V USB" (shape input) (at 26.67 19.05 0) (fields_autoplaced)
+  (hierarchical_label "V USB" (shape input) (at 49.53 79.375 0) (fields_autoplaced)
     (effects (font (size 1.27 1.27)) (justify left))
   )
@@
     )
   )
-  (symbol (lib_id "power:VDD") (at 68.58 111.76 0) (unit 1)
-    (in_bom yes) (on_board yes) (dnp no) (fields_autoplaced)
-    (property "Reference" "#PWR023" (at 68.58 115.57 0)
-      (effects (font (size 1.27 1.27)) hide)
-    )
-    (property "Value" "VDD" (at 68.58 108.188 0)
-      (effects (font (size 1.27 1.27)))
-    )
-    (property "Footprint" "" (at 68.58 111.76 0)
-      (effects (font (size 1.27 1.27)) hide)
-    )
-    (property "Datasheet" "" (at 68.58 111.76 0)
-      (effects (font (size 1.27 1.27)) hide)
-    )
-    (pin "1")
-    (instances
-      (project "DisplayU_Sisterboard"
-        (path "/19c7c935-33c8-4c59-9a5d-d605e15c31a3/25a7bd83-bec9-4f3f-8272-59937481b0db/21567c23-4b19-440e-b334-053946d84a03"
-          (reference "#PWR023") (unit 1)
-        )
-        (path "/19c7c935-33c8-4c59-9a5d-d605e15c31a3/25a7bd83-bec9-4f3f-8272-59937481b0db"
-          (reference "#PWR023") (unit 1)
-        )
-      )
-    )
-  )
-  (symbol (lib_id "power:GND") (at 19.685 24.13 0) (unit 1)
+  (symbol (lib_id "power:VDD") (at 68.58 116.84 0) (unit 1)
+    (in_bom yes) (on_board yes) (dnp no) (fields_autoplaced)
+    (property "Reference" "#PWR023" (at 68.58 120.65 0)
+      (effects (font (size 1.27 1.27)) hide)
+    )
+    (property "Value" "VDD" (at 68.58 113.268 0)
+      (effects (font (size 1.27 1.27)))
+    )
+    (property "Footprint" "" (at 68.58 116.84 0)
+      (effects (font (size 1.27 1.27)) hide)
+    )
+    (property "Datasheet" "" (at 68.58 116.84 0)
+      (effects (font (size 1.27 1.27)) hide)
+    )
+    (pin "1")
+    (instances
+      (project "DisplayU_Sisterboard"
+        (path "/19c7c935-33c8-4c59-9a5d-d605e15c31a3/25a7bd83-bec9-4f3f-8272-59937481b0db/21567c23-4b19-440e-b334-053946d84a03"
+          (reference "#PWR023") (unit 1)
+        )
+        (path "/19c7c935-33c8-4c59-9a5d-d605e15c31a3/25a7bd83-bec9-4f3f-8272-59937481b0db"
+          (reference "#PWR023") (unit 1)
+        )
+      )
+    )
+  )
+  (symbol (lib_id "power:GND") (at 42.545 84.455 0) (unit 1)
     (in_bom yes) (on_board yes) (dnp no)
-    (property "Reference" "#PWR024" (at 19.685 30.48 0)
-      (effects (font (size 1.27 1.27)) hide)
-    )
-    (property "Value" "GND" (at 19.685 27.94 0)
-      (effects (font (size 1.27 1.27)))
-    )
-    (property "Footprint" "" (at 19.685 24.13 0)
-      (effects (font (size 1.27 1.27)) hide)
-    )
-    (property "Datasheet" "" (at 19.685 24.13 0)
+    (property "Reference" "#PWR024" (at 42.545 90.805 0)
+      (effects (font (size 1.27 1.27)) hide)
+    )
+    (property "Value" "GND" (at 42.545 88.265 0)
+      (effects (font (size 1.27 1.27)))
+    )
+    (property "Footprint" "" (at 42.545 84.455 0)
+      (effects (font (size 1.27 1.27)) hide)
+    )
+    (property "Datasheet" "" (at 42.545 84.455 0)
       (effects (font (size 1.27 1.27)) hide)
     )
@@
     )
   )
-  (symbol (lib_id "power:VBUS") (at 26.67 19.05 0) (unit 1)
-    (in_bom yes) (on_board yes) (dnp no) (fields_autoplaced)
-    (property "Reference" "#PWR021" (at 26.67 22.86 0)
-      (effects (font (size 1.27 1.27)) hide)
-    )
-    (property "Value" "VBUS" (at 26.67 15.478 0)
-      (effects (font (size 1.27 1.27)))
-    )
-    (property "Footprint" "" (at 26.67 19.05 0)
-      (effects (font (size 1.27 1.27)) hide)
-    )
-    (property "Datasheet" "" (at 26.67 19.05 0)
+  (symbol (lib_id "power:VBUS") (at 49.53 79.375 0) (unit 1)
+    (in_bom yes) (on_board yes) (dnp no) (fields_autoplaced)
+    (property "Reference" "#PWR021" (at 49.53 83.185 0)
+      (effects (font (size 1.27 1.27)) hide)
+    )
+    (property "Value" "VBUS" (at 49.53 75.803 0)
+      (effects (font (size 1.27 1.27)))
+    )
+    (property "Footprint" "" (at 49.53 79.375 0)
+      (effects (font (size 1.27 1.27)) hide)
+    )
+    (property "Datasheet" "" (at 49.53 79.375 0)
       (effects (font (size 1.27 1.27)) hide)
     )
@@
     )
   )
-  (symbol (lib_id "power:VDD") (at 19.685 19.05 0) (unit 1)
-    (in_bom yes) (on_board yes) (dnp no) (fields_autoplaced)
-    (property "Reference" "#PWR023" (at 19.685 22.86 0)
-      (effects (font (size 1.27 1.27)) hide)
-    )
-    (property "Value" "VDD" (at 19.685 15.478 0)
-      (effects (font (size 1.27 1.27)))
-    )
-    (property "Footprint" "" (at 19.685 19.05 0)
-      (effects (font (size 1.27 1.27)) hide)
-    )
-    (property "Datasheet" "" (at 19.685 19.05 0)
+  (symbol (lib_id "power:VDD") (at 42.545 79.375 0) (unit 1)
+    (in_bom yes) (on_board yes) (dnp no) (fields_autoplaced)
+    (property "Reference" "#PWR023" (at 42.545 83.185 0)
+      (effects (font (size 1.27 1.27)) hide)
+    )
+    (property "Value" "VDD" (at 42.545 75.803 0)
+      (effects (font (size 1.27 1.27)))
+    )
+    (property "Footprint" "" (at 42.545 79.375 0)
+      (effects (font (size 1.27 1.27)) hide)
+    )
+    (property "Datasheet" "" (at 42.545 79.375 0)
       (effects (font (size 1.27 1.27)) hide)
     )
@@
         )
       )
-    )
-  )
-  (symbol (lib_id "Device:R_Small") (at 68.58 113.665 180) (unit 1)
-    (in_bom yes) (on_board yes) (dnp no)
-    (property "Reference" "R1" (at 71.755 112.395 0)
-      (effects (font (size 1.27 1.27)) (justify left))
-    )
-    (property "Value" "4.7k" (at 73.025 114.3 0)
-      (effects (font (size 1.27 1.27)) (justify left))
-    )
-    (property "Footprint" "" (at 68.58 113.665 0)
-      (effects (font (size 1.27 1.27)) hide)
-    )
-    (property "Datasheet" "~" (at 68.58 113.665 0)
-      (effects (font (size 1.27 1.27)) hide)
-    )
-    (pin "1")
-    (pin "2")
-    (instances
-      (project "DisplayU_Sisterboard"
-        (path "/19c7c935-33c8-4c59-9a5d-d605e15c31a3/25a7bd83-bec9-4f3f-8272-59937481b0db/21567c23-4b19-440e-b334-053946d84a03"
-          (reference "R1") (unit 1)
-        )
-        (path "/19c7c935-33c8-4c59-9a5d-d605e15c31a3/25a7bd83-bec9-4f3f-8272-59937481b0db"
-          (reference "R1") (unit 1)
-        )
-      )
