File: KiCad/Production/DisplayU_Sisterboard/Power.kicad_sch (KiCad schematic)
At the start: 17 parts, among them Q2 AO3407, U3 AP2112K-3.3

Commit message: Routing
Parts:
- removed F?: 0.7A, symbol Device:Fuse
- C?: value 0.1uF -> 0.1µ
- C?: value 0.22uF -> 0.22µ
- C?: value 10uF -> 10µ
- D? (x2): footprint (none) -> LED_SMD:LED_0603_1608Metric
- F?: footprint (none) -> Fuse:Fuse_0603_1608Metric
- J?: footprint (none) -> Connector_JST:JST_PH_S2B-PH-SM4-TB_1x02-1MP_P2.00mm_Horizontal
- L?: value 1.5µH -> 1.5µ; footprint (none) -> Inductor_SMD:L_1210_3225Metric
- Q2: value AO3407 -> AO3421E
- U3: value AP2112K-3.3 -> AP2112K-3.3TRG1
- U?: value LTC4001 -> LTC4001EUF#TRPBF
Connections:
- net BATT+: now also Q2.3 (D)
- net GND: no longer F?.2, R?.2
- new net VBAT: F?.2, R?.2
Other:
- note added: "- Sam Dilmaghanian"
- note added: "Datasheet"
Changed lines of the file:
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@@
     (stroke (width 0) (type default))
   )
-  (wire (pts (xy 113.665 105.41) (xy 113.665 104.775))
+  (wire (pts (xy 113.665 112.395) (xy 113.665 113.665))
     (stroke (width 0) (type default))
   )
@@
     (stroke (width 0) (type default))
   )
-  (wire (pts (xy 105.41 82.55) (xy 105.41 80.01))
-    (stroke (width 0) (type default))
-  )
   (wire (pts (xy 165.1 59.69) (xy 165.1 67.31))
     (stroke (width 0) (type default))
@@
   )
   (wire (pts (xy 86.36 78.105) (xy 86.36 80.01))
-    (stroke (width 0) (type default))
-  )
-  (wire (pts (xy 113.665 113.03) (xy 113.665 113.665))
     (stroke (width 0) (type default))
   )
@@
   (text "Connectors" (at 81.28 51.435 0)
     (effects (font (size 1.27 1.27) (thickness 0.254) bold) (justify left bottom))
+  )
+  (text "- Sam Dilmaghanian" (at 212.09 180.34 0)
+    (effects (font (size 1.27 1.27)) (justify left bottom))
   )
   (text "Embedded Bike Safety: Display U Board (Concept)\n" (at 186.055 191.135 0)
@@
     (at 177.8 176.53 0)
     (effects (font (size 1.9 1.9)) (justify left bottom))
+  )
+  (text "Datasheet" (at 193.04 53.975 0)
+    (effects (font (size 1.27 1.27)) (justify left bottom) (href "https://www.analog.com/media/en/technical-documentation/data-sheets/4001f.pdf"))
   )
   (label "Charge" (at 152.4 85.09 0) (fields_autoplaced)
@@
     )
   )
-  (global_label "BATT+" (shape input) (at 113.665 104.775 90) (fields_autoplaced)
-    (effects (font (size 1.27 1.27)) (justify left))
-    (property "Intersheetrefs" "${INTERSHEET_REFS}" (at 113.665 96.8631 90)
+  (global_label "BATT+" (shape input) (at 113.665 112.395 90) (fields_autoplaced)
+    (effects (font (size 1.27 1.27)) (justify left))
+    (property "Intersheetrefs" "${INTERSHEET_REFS}" (at 113.665 104.4831 90)
       (effects (font (size 1.27 1.27)) (justify left) hide)
     )
@@
       (effects (font (size 1.27 1.27)) (justify left))
     )
-    (property "Footprint" "" (at 91.44 62.23 0)
+    (property "Footprint" "Connector_JST:JST_PH_S2B-PH-SM4-TB_1x02-1MP_P2.00mm_Horizontal" (at 91.44 62.23 0)
       (effects (font (size 1.27 1.27)) hide)
     )
@@
     )
   )
-  (symbol (lib_id "power:GND") (at 105.41 82.55 0) (unit 1)
-    (in_bom yes) (on_board yes) (dnp no) (fields_autoplaced)
-    (property "Reference" "#PWR?" (at 105.41 88.9 0)
-      (effects (font (size 1.27 1.27)) hide)
-    )
-    (property "Value" "GND" (at 105.41 86.9934 0)
-      (effects (font (size 1.27 1.27)))
-    )
-    (property "Footprint" "" (at 105.41 82.55 0)
-      (effects (font (size 1.27 1.27)) hide)
-    )
-    (property "Datasheet" "" (at 105.41 82.55 0)
-      (effects (font (size 1.27 1.27)) hide)
-    )
-    (pin "1")
-    (instances
-      (project "EBS_Main"
-        (path "/0a240a99-769c-44e4-a1cf-c8ae622a9801/bdd1c018-ef1f-4016-b07d-24e58036b989"
-          (reference "#PWR?") (unit 1)
-        )
-      )
-      (project "DisplayU_Sisterboard"
-        (path "/19c7c935-33c8-4c59-9a5d-d605e15c31a3/bc90aa39-2744-4a84-88b0-6b5f6472e99d"
-          (reference "#PWR035") (unit 1)
-        )
-      )
-    )
-  )
   (symbol (lib_id "Device:C") (at 170.815 80.01 90) (unit 1)
     (in_bom yes) (on_board yes) (dnp no)
@@
       (effects (font (size 1.27 1.27)))
     )
-    (property "Value" "0.1uF" (at 172.72 83.82 90)
+    (property "Value" "0.1µ" (at 172.72 83.82 90)
       (effects (font (size 1.27 1.27)))
     )
@@
   (symbol (lib_id "Battery_Management:LTC4001") (at 191.77 69.85 0) (unit 1)
     (in_bom yes) (on_board yes) (dnp no)
-    (property "Reference" "U?" (at 193.7894 50.9102 0)
-      (effects (font (size 1.27 1.27)) (justify left))
-    )
-    (property "Value" "LTC4001" (at 193.7894 53.4471 0)
+    (property "Reference" "U?" (at 193.04 47.6281 0)
+      (effects (font (size 1.27 1.27)) (justify left))
+    )
+    (property "Value" "LTC4001EUF#TRPBF\n" (at 193.04 50.165 0)
       (effects (font (size 1.27 1.27)) (justify left))
     )
@@
       (effects (font (size 1.27 1.27)))
     )
-    (property "Value" "0.22uF" (at 172.085 64.135 90)
+    (property "Value" "0.22µ" (at 172.085 64.135 90)
       (effects (font (size 1.27 1.27)))
     )
@@
       (effects (font (size 1.27 1.27)) (justify right))
     )
-    (property "Footprint" "" (at 133.35 68.58 0)
+    (property "Footprint" "LED_SMD:LED_0603_1608Metric" (at 133.35 68.58 0)
       (effects (font (size 1.27 1.27)) hide)
     )
@@
       (effects (font (size 1.27 1.27)) (justify left))
     )
-    (property "Value" "AO3407" (at 116.205 118.745 0)
+    (property "Value" "AO3421E\n" (at 116.205 118.745 0)
       (effects (font (size 1.27 1.27)) (justify left))
     )
@@
       (effects (font (size 1.27 1.27)))
     )
-    (property "Value" "1.5µH" (at 208.28 58.0256 90)
-      (effects (font (size 1.27 1.27)))
-    )
-    (property "Footprint" "" (at 208.28 59.69 0)
+    (property "Value" "1.5µ" (at 208.28 58.0256 90)
+      (effects (font (size 1.27 1.27)))
+    )
+    (property "Footprint" "Inductor_SMD:L_1210_3225Metric" (at 208.28 59.69 0)
       (effects (font (size 1.27 1.27)) hide)
     )
@@
   (symbol (lib_id "Regulator_Linear:AP2112K-3.3") (at 131.445 130.175 0) (unit 1)
     (in_bom yes) (on_board yes) (dnp no) (fields_autoplaced)
-    (property "Reference" "U3" (at 131.445 120.65 0)
-      (effects (font (size 1.27 1.27)))
-    )
-    (property "Value" "AP2112K-3.3" (at 131.445 123.19 0)
+    (property "Reference" "U3" (at 131.445 122.0658 0)
+      (effects (font (size 1.27 1.27)))
+    )
+    (property "Value" "AP2112K-3.3TRG1\n" (at 131.445 124.571 0)
       (effects (font (size 1.27 1.27)))
     )
@@
   (symbol (lib_id "Device:C") (at 220.98 76.2 0) (unit 1)
     (in_bom yes) (on_board yes) (dnp no) (fields_autoplaced)
-    (property "Reference" "C?" (at 223.901 75.3653 0)
-      (effects (font (size 1.27 1.27)) (justify left))
-    )
-    (property "Value" "10uF" (at 223.901 77.9022 0)
+    (property "Reference" "C?" (at 223.901 75.3752 0)
+      (effects (font (size 1.27 1.27)) (justify left))
+    )
+    (property "Value" "10µ" (at 223.901 77.8804 0)
       (effects (font (size 1.27 1.27)) (justify left))
     )
@@
       (effects (font (size 1.27 1.27)))
     )
-    (property "Footprint" "" (at 96.52 81.788 90)
+    (property "Footprint" "Fuse:Fuse_0603_1608Metric" (at 96.52 81.788 90)
       (effects (font (size 1.27 1.27)) hide)
     )
@@
       (effects (font (size 1.27 1.27)) (justify right))
     )
-    (property "Footprint" "" (at 152.4 81.28 0)
+    (property "Footprint" "LED_SMD:LED_0603_1608Metric" (at 152.4 81.28 0)
       (effects (font (size 1.27 1.27)) hide)
     )
@@
         )
       )
-    )
-  )
-  (symbol (lib_id "Device:Fuse") (at 113.665 109.22 0) (unit 1)
-    (in_bom yes) (on_board yes) (dnp no) (fields_autoplaced)
-    (property "Reference" "F?" (at 115.189 107.9575 0)
-      (effects (font (size 1.27 1.27)) (justify left))
-    )
-    (property "Value" "0.7A" (at 115.189 110.4825 0)
-      (effects (font (size 1.27 1.27)) (justify left))
-    )
-    (property "Footprint" "" (at 111.887 109.22 90)
-      (effects (font (size 1.27 1.27)) hide)
-    )
-    (property "Datasheet" "~" (at 113.665 109.22 0)
-      (effects (font (size 1.27 1.27)) hide)
-    )
-    (pin "1")
-    (pin "2")
-    (instances
-      (project "EBS_Main"
-        (path "/0a240a99-769c-44e4-a1cf-c8ae622a9801/bdd1c018-ef1f-4016-b07d-24e58036b989"
-          (reference "F?") (unit 1)
-        )
-      )
-      (project "DisplayU_Sisterboard"
-        (path "/19c7c935-33c8-4c59-9a5d-d605e15c31a3/bc90aa39-2744-4a84-88b0-6b5f6472e99d"
-          (reference "F1") (unit 1)
-        )
-      )

Commit message: Berekening/Metingen Verslag
Parts:
- J?: value JS2 XH 2.5 -> S2B-PH-SM4-TB(LF)(SN)
Changed lines of the file:
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@@
   (symbol (lib_id "Connector:Conn_01x02_Female") (at 91.44 62.23 0) (unit 1)
     (in_bom yes) (on_board yes) (dnp no) (fields_autoplaced)
-    (property "Reference" "J?" (at 92.1512 62.6653 0)
+    (property "Reference" "J?" (at 92.1512 62.6752 0)
       (effects (font (size 1.27 1.27)) (justify left))
     )
-    (property "Value" "JS2 XH 2.5" (at 92.1512 65.2022 0)
+    (property "Value" "S2B-PH-SM4-TB(LF)(SN)" (at 92.1512 65.1804 0)
       (effects (font (size 1.27 1.27)) (justify left))
     )
