File: KiCad/Production/DisplayU_Sisterboard/DisplayU_Sisterboard.kicad_pcb (KiCad board)
At the start: 2 copper layers, 40 parts, among them J1 USB_C_Plug_USB2.0, Q1 FDS9926A, Q2 FDS9926A, U3 AP9101CK, U4 LTC4001

Commit message: Routing
Parts:
- removed C11: 100nF, Capacitor_SMD:C_0603_1608Metric_Pad1.08x0.95mm_HandSolder
- removed C8: 10uF, Capacitor_SMD:C_0603_1608Metric_Pad1.08x0.95mm_HandSolder
- removed C9: 22uF, Capacitor_SMD:C_0603_1608Metric
- removed D1: Debug, Diode_SMD:D_0603_1608Metric
- removed R8: 1k, Resistor_SMD:R_0603_1608Metric
- added D10: C_Fault, LED_SMD:LED_0603_1608Metric, F.Cu at (-14.9, 237.4)
- added D12: PLED, LED_SMD:LED_0603_1608Metric, F.Cu at (-19.9, 237.4)
- added D2: XPEBRD-L1-0000-00901, VUBRacing_ELO:XPEBRD-L1-0000-00901, F.Cu at (-75.8, 230.1)
- added D3: XPEBRD-L1-0000-00901, VUBRacing_ELO:XPEBRD-L1-0000-00901, F.Cu at (-4.64, 237.7)
- added D4: BZT52C5V6S-7-F, Diode_SMD:D_SOD-323F, F.Cu at (-59.5, 224.8)
- added D5: 1N5819, Diode_SMD:D_SOD-323F, F.Cu at (-32.1, 229.4)
- added F1: 04941.25NRHF, Fuse:Fuse_0603_1608Metric, F.Cu at (-28.6, 218.5)
- added F5: 3A, Fuse:Fuse_0603_1608Metric, F.Cu at (-12.8, 224.0)
- added J2: USB-C USB 2.0 MC-372, VUBRacing_ELO:USB C 2.0 MC 772, F.Cu at (-62.1, 207.7)
- added L1: 4.7n ±5%, Inductor_SMD:L_0603_1608Metric, F.Cu at (-45.9, 227.4)
- added L2: 2.2n ±5%, Inductor_SMD:L_0603_1608Metric, F.Cu at (-45.9, 230.5)
- added L3: 10µ, Inductor_SMD:L_0603_1608Metric, F.Cu at (-36.8, 220.4)
- added L4: 15n, Inductor_SMD:L_0603_1608Metric, F.Cu at (-36.7, 222.0)
- added L5: 1.5µ, Inductor_SMD:L_1210_3225Metric, F.Cu at (-26.9, 224.2)
- added R6: 820K, Resistor_SMD:R_0603_1608Metric, F.Cu at (-13.5, 221.4)
- added R7: 2M, Resistor_SMD:R_0603_1608Metric, F.Cu at (-16.6, 221.4)
- added REF**: MountingHole_2.7mm_M2.5, MountingHole:MountingHole_2.7mm_M2.5, F.Cu at (-19.0, 214.0)
- added REF**: MountingHole_2.7mm_M2.5, MountingHole:MountingHole_2.7mm_M2.5, F.Cu at (-55.0, 235.0)
- added REF**: MountingHole_2.7mm_M2.5, MountingHole:MountingHole_2.7mm_M2.5, F.Cu at (-76.0, 214.0)
- added RST1: Jumper_2_Open, Button_Switch_SMD:SW_SPST_B3U-1000P, F.Cu at (-52.3, 219.6)
- added TP1: TestPoint, TestPoint:TestPoint_Pad_D2.0mm, F.Cu at (-48.1, 213.4)
- added X1: 32MHz ±40 ppm, Crystal:Crystal_SMD_SeikoEpson_FA128-4Pin_2.0x1.6mm, F.Cu at (-41.4, 227.2)
- added kibuzzard-64865EC8: G***, kibuzzard-64865EC8, F.Cu at (-19.9, 234.1)
- added kibuzzard-64865EDB: G***, kibuzzard-64865EDB, F.Cu at (-14.9, 234.1)
- added kibuzzard-64865F18: G***, kibuzzard-64865F18, F.Cu at (-76.0, 230.8)
- added kibuzzard-64865F2D: G***, kibuzzard-64865F2D, F.Cu at (-4.50, 230.6)
- added kibuzzard-6486612E: G***, kibuzzard-6486612E, F.Cu at (-70.5, 220.0)
- added kibuzzard-64866148: G***, kibuzzard-64866148, F.Cu at (-75.8, 222.6)
- added kibuzzard-64866152: G***, kibuzzard-64866152, F.Cu at (-77.2, 224.9)
- C12: value 0.22uF -> 0.22µ
- C13: value 0.1uF -> 0.1µ
- C14: value 10uF -> 10µ
- J1: value USB_C_Plug_USB2.0 -> JS2 XH 2.5; footprint Connector_USB:USB_C_Receptacle_GCT_USB4135-GF-A_6P_TopMnt_Horizontal -> Connector_JST:JST_PH_S2B-PH-SM4-TB_1x02-1MP_P2.00mm_Horizontal
- Q2: value FDS9926A -> AO3421E; footprint Package_SO:SOIC-8_3.9x4.9mm_P1.27mm -> Package_TO_SOT_SMD:SOT-23
- R11: value 330 -> 5.1K
- R12: value 2.7k -> 100K
- R2, R3: value R -> CHP1206AFX-47R0ELF
- R9: value 1k -> 5.1K
- U3: value AP9101CK -> AP2112K-3.3TRG1
- U4: value LTC4001 -> LTC4001EUF#TRPBF
- moved U1 277.3 mm to (-42.6, 220.8), turned to -90 degrees
- moved C21 262.0 mm to (-59.4, 223.0)
- moved C6 255.9 mm to (-40.6, 230.2), turned to -90 degrees
- moved C7 255.1 mm to (-42.1, 230.2), turned to -90 degrees
- moved C20 254.9 mm to (-47.4, 223.3), turned to 180 degrees
- moved C19 253.3 mm to (-47.4, 218.4), turned to 180 degrees
- moved AE1 252.6 mm to (-46.0, 232.7), turned to 180 degrees
- moved C3 252.2 mm to (-47.6, 227.4), turned to 90 degrees
- moved C16 250.9 mm to (-44.1, 227.4), turned to -90 degrees
- moved C18 249.5 mm to (-43.3, 214.6), turned to 90 degrees
- moved R9 246.8 mm to (-63.1, 223.0), turned to 180 degrees
- moved C2 246.5 mm to (-36.7, 227.2)
- moved R11 245.5 mm to (-66.2, 223.0)
- moved C1 242.6 mm to (-41.6, 214.6), turned to 90 degrees
- moved C4 241.5 mm to (-36.7, 225.4)
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Connections:
- net Net-(U1-XC1) renamed /MCU & Comms/MicroController/X1-
- net Net-(U1-XC2) renamed /MCU & Comms/MicroController/X1+
- C1 pad 1: +3.3V -> VDD
- C10 pad 1: +5V -> VBUS
- C14 pad 1: +BATT -> BATT+
- C15 pad 1: +3.3V -> VDD
- C18 pad 1: +3.3V -> VDD
- C20 pad 1: +3.3V -> VDD
- Q2 pad 1: GND -> VBUS
- Q2 pad 2: Net-(Q2A-G1) -> Net-(D5-K)
- Q2 pad 3: GND -> BATT+
- R11 pad 1: Net-(U3-VDD) -> CC2
- R11 pad 2: +BATT -> GND
- R12 pad 1: Net-(U3-VM) -> VBUS
- R13 pad 2: +5V -> VBAT
- R2 pad 1: VCC -> VBAT
- R3 pad 1: VCC -> VBAT
- R9 pad 1: Net-(D9-K) -> CC1
- U1 pad 12: /D- -> DATA-
- U1 pad 13: /D+ -> DATA+
- U1 pad 16: +3.3V -> /MCU & Comms/MicroController/RST
- U1 pad 18: +3.3V -> VDD
- U1 pad 30: +3.3V -> VDD
- U1 pad 31: unconnected-(U1-P0.08-Pad31) -> (no net)
- U1 pad 4: /MCU & Comms/MicroController/IO 2 -> Charge Fault
- U1 pad 40: +3.3V -> Net-(F1-Pad1)
- U1 pad 6: /MCU & Comms/MicroController/IO 4 -> Charge Status
- U1 pad 8: +3.3V -> VDD
- U1 pad 9: +3.3V -> VDD
- U3 pad 1: Net-(U3-VM) -> Net-(D5-K)
- U3 pad 2: Net-(U3-VDD) -> GND
- U3 pad 3: GND -> Net-(D5-K)
- U3 pad 4: Net-(Q2B-G2) -> unconnected-(U3-NC-Pad4)
- U3 pad 5: Net-(Q2A-G1) -> VDD
- U4 pad 1: +BATT -> BATT+
- U4 pad 10: /Power Electronics/C_Fault -> Charge Fault
- U4 pad 16: +BATT -> BATT+
- U4 pad 7: /Power Electronics/Charge -> Charge Status
- U4 pad 8: +5V -> VBUS
- U4 pad 9: +5V -> VBUS
Routing:
- net VBUS: track 0.00 -> 119.5 mm, vias 0 -> 5
- net Net-(D2-Pad1): track 0.00 -> 70.9 mm, vias 0 -> 2
- net Net-(D2-Pad2): track 0.00 -> 62.6 mm, vias 0 -> 2
- net Net-(D3-Pad2): track 0.00 -> 60.0 mm
- net VDD: track 0.00 -> 53.3 mm, vias 0 -> 5
- net /MCU & Comms/MicroController/IO 3: track 0.00 -> 46.1 mm, vias 0 -> 2
- net Charge Fault: track 0.00 -> 42.0 mm, vias 0 -> 3
- net Charge Status: track 0.00 -> 41.9 mm, vias 0 -> 3
- net BATT+: track 0.00 -> 31.9 mm
- net DATA+: track 0.00 -> 23.3 mm, vias 0 -> 2
- net DATA-: track 0.00 -> 22.7 mm
- net Net-(F1-Pad1): track 0.00 -> 20.8 mm
- net Net-(D5-K): track 0.00 -> 17.4 mm
- net /MCU & Comms/Right: track 0.00 -> 14.2 mm
- net VBAT: track 0.00 -> 14.2 mm
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- added copper zone on B.Cu, net /MCU & Comms/Left
- added copper zone on F.Cu, net /MCU & Comms/Left
- added copper zone on B.Cu, net /MCU & Comms/MicroController/IO 3
- added copper zone on F.Cu, net /MCU & Comms/MicroController/IO 3
- added copper zone on B.Cu, net /MCU & Comms/MicroController/IO 5
- added copper zone on F.Cu, net /MCU & Comms/MicroController/IO 5
- added copper zone on B.Cu, net /MCU & Comms/MicroController/RST
- added copper zone on F.Cu, net /MCU & Comms/MicroController/RST
- added copper zone on F.Cu, net BATT+
- added copper zone on B.Cu, net CC1
- added copper zone on F.Cu, net CC1
- added copper zone on B.Cu, net Charge Fault
- added copper zone on F.Cu, net Charge Fault
- added copper zone on B.Cu, net Charge Status
- added copper zone on F.Cu, net Charge Status
- added copper zone on B.Cu, net DATA+
- added copper zone on F.Cu, net DATA+
- added copper zone on B.Cu, net GND
- added copper zone on F.Cu, net GND
- added copper zone on B.Cu, net Net-(D2-Pad1)
- added copper zone on F.Cu, net Net-(D2-Pad1)
- added copper zone on B.Cu, net Net-(D2-Pad2)
- added copper zone on F.Cu, net Net-(D2-Pad2)
- added copper zone on B.Cu, net Net-(U1-ANT_RF)
- added copper zone on F.Cu, net Net-(U1-ANT_RF)
- added copper zone on B.Cu, net Net-(U1-DEC4)
- added copper zone on F.Cu, net Net-(U1-DEC4)
- added copper zone on B.Cu, net VBUS
- added copper zone on F.Cu, net VBUS
- added copper zone on B.Cu, net VDD
- added copper zone on F.Cu, net VDD
Other:
- board outline added: 80 x 28.4 mm
- board text added: "Ingebedde DSP-systemen Vrije Universiteit Brussel 06/2023 Sam Dilmaghanian"
- board text added: "P0.07"

Commit message: Fixes
Parts:
- moved C6 0.41 mm to (-40.6, 229.8)
- moved C7 0.41 mm to (-42.1, 229.8)
- moved X1 0.41 mm to (-41.4, 226.8)
- renumbered RST1 to RST
Routing:
- net GND: vias 11 -> 12

Commit message: Documentation&3DCAD
Parts:
- added kibuzzard-648A3F17: G***, kibuzzard-648A3F17, F.Cu at (-61.8, 203.2)
- added kibuzzard-648A3F39: G***, kibuzzard-648A3F39, F.Cu at (-61.9, 205.1)
- added kibuzzard-648A3F78: G***, kibuzzard-648A3F78, F.Cu at (-67.0, 209.8)
- moved REF** 62.0 mm to (-136.9, 202.5)
- moved kibuzzard-64866148 62.0 mm to (-136.7, 211.0)
- moved C6 62.0 mm to (-101.5, 218.3)
- moved C7 62.0 mm to (-103.0, 218.3)
- moved L3 62.0 mm to (-97.7, 208.8)
- moved L5 62.0 mm to (-87.8, 212.7)
- moved R13 62.0 mm to (-80.9, 224.0)
- moved R7 62.0 mm to (-77.6, 209.9)
- moved RST 62.0 mm to (-113.2, 208.1)
- moved kibuzzard-64865EC8 62.0 mm to (-80.8, 222.6)
- moved kibuzzard-64865EDB 62.0 mm to (-75.8, 222.6)
- moved AE1 62.0 mm to (-107.0, 221.2)
- moved C1 62.0 mm to (-102.6, 203.1)
- moved C10 62.0 mm to (-91.0, 221.3)
- moved C12 62.0 mm to (-82.6, 216.3)
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
Commit message: Logo EBS
Parts:
- added G***: LOGO, LOGO, F.Cu at (-127.7, 221.2)
