File: KiCad/Production/SenseU_Mainboard/nRF52820.kicad_sch (KiCad schematic)
At the start: 0 parts

Commit message: added a lot
Parts:
- added C1, C4: 1µ, Capacitor_SMD:C_0603_1608Metric, symbol Device:C_Small
- added C15, C17, C20: 100n, Capacitor_SMD:C_0603_1608Metric, symbol Device:C_Small
- added C16: 100p ±5%, Capacitor_SMD:C_0603_1608Metric, symbol Device:C_Small
- added C18, C19, C21: 4.7µ, Capacitor_SMD:C_0603_1608Metric, symbol Device:C_Small
- added C2: 1p ±2%, Capacitor_SMD:C_0603_1608Metric, symbol Device:C_Small
- added C3: 1.2p ±5%, Capacitor_SMD:C_0603_1608Metric, symbol Device:C_Small
- added C5: 47n, Capacitor_SMD:C_0603_1608Metric, symbol Device:C_Small
- added C6, C7: 12p ±2%, Capacitor_SMD:C_0603_1608Metric, symbol Device:C_Small
- added F?: 04941.25NRHF, Fuse:Fuse_0603_1608Metric, symbol Device:Fuse
- added L1: 4.7n ±5%, Inductor_SMD:L_0603_1608Metric, symbol Device:L_Small
- added L2: 2.2n ±5%, Inductor_SMD:L_0603_1608Metric, symbol Device:L_Small
- added L3: 10µ, Inductor_SMD:L_0603_1608Metric, symbol Device:L_Small
- added L4: 15n, Inductor_SMD:L_0603_1608Metric, symbol Device:L_Small
- added U1: ~, Package_DFN_QFN:QFN-40-1EP_5x5mm_P0.4mm_EP3.8x3.8mm, symbol NRF:nRF52820
- added X1: 32MHz ±40 ppm, Crystal:Crystal_SMD_SeikoEpson_FA128-4Pin_2.0x1.6mm, symbol Device:Crystal_Small
Connections:
- new net: C17.1, U1.1 (DEC1)
- new net: C19.1, U1.11 (DECUSB)
- new net: C2.1, L1.1, U1.24 (ANT_RF)
- new net: C4.1, C5.1, L4.1, U1.26 (DEC6), U1.38 (DEC4)
- new net: C16.1, U1.27 (DEC3)
- new net: L3.2, U1.39 (DCC)
- new net: F?.1, U1.40 (VDD)
- new net: L3.1, L4.2
- new net: C3.1, L1.2, L2.1
- new net DATA+: U1.13 (D+_USB)
- new net DATA-: U1.12 (D-_USB)
- new net GND: C1.2, C15.2, C16.2, C17.2, C18.2, C19.2, C2.2, C20.2, C21.2, C3.2, C4.2, C5.2, C6.2, C7.2, U1.25 (VSS_PA), U1.37 (VSS), U1.41 (VSS)
- new net IO 0: U1.2 (P0.00/XL1)
- new net IO 1: U1.3 (P0.01/XL2)
- new net IO 2: U1.4 (P0.04_AIN2)
- new net IO 3: U1.5 (P0.05_AIN3)
- new net IO 4: U1.6 (P0.06)
- new net IO 5: U1.7 (P0.07)
- new net IO 6: U1.31 (P0.08)
- new net RF: L2.2
- new net RST: U1.16 (P0.18/RST)
- new net VBUS: C21.1, U1.10 (VBUS)
- new net VDD: C1.1, C15.1, C18.1, C20.1, F?.2, U1.18 (VDD), U1.30 (VDD), U1.8 (VDD), U1.9 (VDDH)
- new net X1+: C6.1, U1.29 (XC2), X1.2
- new net X1-: C7.1, U1.28 (XC1), X1.1
Other:
- note added: "Datasheet"
- note added: "VDD: Battery USB: Enabled"
