File: KiCad/Production/SenseU_Mainboard/USB2UART.kicad_sch (KiCad schematic)
At the start: 3 parts, among them U4 COM-16278

Commit message: assigning components
Parts:
- renumbered C20 to C21, C19 to C22, U4 to U5
Changed lines of the file:
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@@
   (symbol (lib_id "CH340:COM-16278") (at 109.22 129.54 0) (unit 1)
     (in_bom yes) (on_board yes) (dnp no) (fields_autoplaced)
-    (property "Reference" "U4" (at 109.22 110.998 0)
+    (property "Reference" "U5" (at 109.22 110.998 0)
       (effects (font (size 1.27 1.27)))
     )
@@
       (project "SenseU_Mainboard"
         (path "/43872b54-cf9c-4c7b-870d-631baccef0c0/d8d785fb-fd90-4cd9-a47e-213577f6aaa3"
-          (reference "U4") (unit 1)
+          (reference "U5") (unit 1)
         )
       )
@@
   (symbol (lib_id "power:GND") (at 127 144.78 0) (unit 1)
     (in_bom yes) (on_board yes) (dnp no) (fields_autoplaced)
-    (property "Reference" "#PWR073" (at 127 151.13 0)
+    (property "Reference" "#PWR069" (at 127 151.13 0)
       (effects (font (size 1.27 1.27)) hide)
     )
@@
       (project "SenseU_Mainboard"
         (path "/43872b54-cf9c-4c7b-870d-631baccef0c0/d8d785fb-fd90-4cd9-a47e-213577f6aaa3"
-          (reference "#PWR073") (unit 1)
+          (reference "#PWR069") (unit 1)
         )
       )
@@
   (symbol (lib_id "Device:C") (at 149.86 120.65 0) (unit 1)
     (in_bom yes) (on_board yes) (dnp no) (fields_autoplaced)
-    (property "Reference" "C19" (at 153.67 120.015 0)
+    (property "Reference" "C22" (at 153.67 120.015 0)
       (effects (font (size 1.27 1.27)) (justify left))
     )
@@
       (project "SenseU_Mainboard"
         (path "/43872b54-cf9c-4c7b-870d-631baccef0c0/d8d785fb-fd90-4cd9-a47e-213577f6aaa3"
-          (reference "C19") (unit 1)
+          (reference "C22") (unit 1)
         )
       )
@@
   (symbol (lib_id "power:GND") (at 139.7 127 0) (unit 1)
     (in_bom yes) (on_board yes) (dnp no) (fields_autoplaced)
-    (property "Reference" "#PWR072" (at 139.7 133.35 0)
+    (property "Reference" "#PWR070" (at 139.7 133.35 0)
       (effects (font (size 1.27 1.27)) hide)
     )
@@
       (project "SenseU_Mainboard"
         (path "/43872b54-cf9c-4c7b-870d-631baccef0c0/d8d785fb-fd90-4cd9-a47e-213577f6aaa3"
-          (reference "#PWR072") (unit 1)
+          (reference "#PWR070") (unit 1)
         )
       )
@@
   (symbol (lib_id "Device:C") (at 139.7 123.19 0) (unit 1)
     (in_bom yes) (on_board yes) (dnp no) (fields_autoplaced)
-    (property "Reference" "C20" (at 143.51 122.555 0)
+    (property "Reference" "C21" (at 143.51 122.555 0)
       (effects (font (size 1.27 1.27)) (justify left))
     )
@@
       (project "SenseU_Mainboard"
         (path "/43872b54-cf9c-4c7b-870d-631baccef0c0/d8d785fb-fd90-4cd9-a47e-213577f6aaa3"
-          (reference "C20") (unit 1)
+          (reference "C21") (unit 1)
         )
       )

Commit message: changed place of usb to uart
Parts:
- C21, C22: footprint (none) -> Capacitor_SMD:C_0603_1608Metric_Pad1.08x0.95mm_HandSolder
Changed lines of the file:
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@@
       (effects (font (size 1.27 1.27)) (justify left))
     )
-    (property "Footprint" "" (at 150.8252 124.46 0)
+    (property "Footprint" "Capacitor_SMD:C_0603_1608Metric_Pad1.08x0.95mm_HandSolder" (at 150.8252 124.46 0)
       (effects (font (size 1.27 1.27)) hide)
     )
@@
       (effects (font (size 1.27 1.27)) (justify left))
     )
-    (property "Footprint" "" (at 140.6652 127 0)
+    (property "Footprint" "Capacitor_SMD:C_0603_1608Metric_Pad1.08x0.95mm_HandSolder" (at 140.6652 127 0)
       (effects (font (size 1.27 1.27)) hide)
     )
