File: KiCad/Production/SenseU_Mainboard/SenseU_Mainboard.kicad_sch (KiCad schematic)
At the start: 5 parts, among them J2 USB-C USB 2.0 MC-372

Commit message: added USB TO UART
Other:
- added sheet USB to UART (USB2UART.kicad_sch)
Changed lines of the file:
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@@
     )
   )
-  (sheet (at 139.7 94.234) (size 32.258 26.416) (fields_autoplaced)
+  (sheet (at 159.004 73.914) (size 32.258 26.416) (fields_autoplaced)
     (stroke (width 0.1524) (type solid))
     (fill (color 0 0 0 0.0000))
-    (property "Sheetname" "Power" (at 139.7 93.5224 0)
+    (property "Sheetname" "Power" (at 159.004 73.2024 0)
       (effects (font (size 1.27 1.27)) (justify left bottom))
     )
-    (property "Sheetfile" "Power.kicad_sch" (at 139.7 121.2346 0)
+    (property "Sheetfile" "Power.kicad_sch" (at 159.004 100.9146 0)
       (effects (font (size 1.27 1.27)) (justify left top))
     )
@@
     )
   )
-  (sheet (at 140.208 57.912) (size 32.258 25.908) (fields_autoplaced)
+  (sheet (at 159.512 37.592) (size 32.258 25.908) (fields_autoplaced)
     (stroke (width 0.1524) (type solid))
     (fill (color 0 0 0 0.0000))
-    (property "Sheetname" "MCU & Comms" (at 140.208 57.2004 0)
+    (property "Sheetname" "MCU & Comms" (at 159.512 36.8804 0)
       (effects (font (size 1.27 1.27)) (justify left bottom))
     )
-    (property "Sheetfile" "MCUnrf.kicad_sch" (at 140.208 84.4046 0)
+    (property "Sheetfile" "MCUnrf.kicad_sch" (at 159.512 64.0846 0)
       (effects (font (size 1.27 1.27)) (justify left top))
     )
@@
       )
     )
+  )
+  (sheet (at 159.258 111.506) (size 25.4 26.924) (fields_autoplaced)
+    (stroke (width 0.1524) (type solid))
+    (fill (color 0 0 0 0.0000))
+    (property "Sheetname" "USB to UART" (at 159.258 110.7944 0)
+      (effects (font (size 1.27 1.27)) (justify left bottom))
+    )
+    (property "Sheetfile" "USB2UART.kicad_sch" (at 159.258 139.0146 0)
+      (effects (font (size 1.27 1.27)) (justify left top))
+    )
+    (instances
+      (project "SenseU_Mainboard"
+        (path "/43872b54-cf9c-4c7b-870d-631baccef0c0" (page "7"))
+      )
+    )

Commit message: routing SenseU done
Parts:
- C?: footprint Capacitor_SMD:C_0603_1608Metric_Pad1.08x0.95mm_HandSolder -> Capacitor_SMD:C_0603_1608Metric
- J2: footprint VUBRacing_ELO:USB C 2.0 MC 772 -> USB_C:GCT_USB4105-GF-A
Other:
- removed sheet USB to UART
Changed lines of the file:
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@@
       (effects (font (size 1.27 1.27)))
     )
-    (property "Footprint" "VUBRacing_ELO:USB C 2.0 MC 772" (at 92.5068 64.008 0)
+    (property "Footprint" "USB_C:GCT_USB4105-GF-A" (at 92.5068 64.008 0)
       (effects (font (size 1.27 1.27)) hide)
     )
@@
       (effects (font (size 1.27 1.27)) (justify left))
     )
-    (property "Footprint" "Capacitor_SMD:C_0603_1608Metric_Pad1.08x0.95mm_HandSolder" (at 68.5292 98.933 0)
+    (property "Footprint" "Capacitor_SMD:C_0603_1608Metric" (at 68.5292 98.933 0)
       (effects (font (size 1.27 1.27)) hide)
     )
@@
       )
     )
-  )
-  (sheet (at 159.258 111.506) (size 25.4 26.924) (fields_autoplaced)
-    (stroke (width 0.1524) (type solid))
-    (fill (color 0 0 0 0.0000))
-    (property "Sheetname" "USB to UART" (at 159.258 110.7944 0)
-      (effects (font (size 1.27 1.27)) (justify left bottom))
-    )
-    (property "Sheetfile" "USB2UART.kicad_sch" (at 159.258 139.0146 0)
-      (effects (font (size 1.27 1.27)) (justify left top))
-    )
-    (instances
-      (project "SenseU_Mainboard"
-        (path "/43872b54-cf9c-4c7b-870d-631baccef0c0" (page "7"))
-      )
-    )
