File: KiCad/Production/SenseU_Mainboard/SenseU_Mainboard.kicad_pcb (KiCad board)
At the start: 2 copper layers, 98.1 x 53.9 mm, 61 parts, among them J1 USB-C USB 2.0 MC-372, J2 JS2 XH 2.5, J3 5-534206-6, J4 1717254-4, Q1 AO3421E, U1 AP2112K-3.3TRG1, U2 LTC4001EUF#TRPBF, U3 COM-16278, X1 32MHz ±40 ppm

Commit message: Logo EBS
Parts:
- added G***: LOGO, LOGO, F.Cu at (174.2, 138.2)
- added H3: MountingHole_2.7mm_M2.5, MountingHole:MountingHole_2.7mm_M2.5, F.Cu at (190.6, 142.2)
- moved H1 10.3 mm to (120.9, 142.3)
